File: trackball-base/buttons.kicad_sch (KiCad schematic)
At the start: 12 parts, among them SW401 D2FC-F-7N, SW402 D2FC-F-7N, SW403 D2FC-F-7N

Commit message: base schematic complete: root + 5 sheets ERC-clean, review notes + BOM draft
Full hierarchical project (root + power/mcu/sensors/buttons/tx):
0 ERC errors, 1 benign pin_to_pin warning (ADC rail-sense, documented).
Netlist-verified: 145 comps, VSEN_1V9/MCU_RST/USB/SPI/TX nets.
Adds notes/SCHEMATIC_REVIEW.md (decisions, rail design, TX tree,
antenna, GPIO map, provisionals, ERC log) + notes/BOM_DRAFT.md.
Other:
- note added: "+3V3/GND join by name; drivers on power sheet"
- note removed: "rail flag: driver on power sheet"
Changed lines of the file:
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@@
     (on_board yes)
     (fields_autoplaced yes)
-    (property "Reference" "#PWR01"
+    (property "Reference" "#PWR301"
       (at 116.84 132.08 0)
       (effects (font (size 1.27 1.27)) hide)
@@
     (on_board yes)
     (fields_autoplaced yes)
-    (property "Reference" "#PWR02"
+    (property "Reference" "#PWR302"
       (at 144.78 115.57 0)
       (effects (font (size 1.27 1.27)) hide)
@@
   )
   (wire
-    (pts (xy 149.86 134.62) (xy 149.86 137.16))
-    (stroke (width 0) (type default))
-  )
-  (symbol
-    (lib_id "power:PWR_FLAG")
-    (at 149.86 137.16 0)
-    (unit 1)
-    (exclude_from_sim no)
-    (in_bom yes)
-    (on_board yes)
-    (fields_autoplaced yes)
-    (property "Reference" "#PWR03"
-      (at 149.86 137.16 0)
-      (effects (font (size 1.27 1.27)) hide)
-    )
-    (property "Value" "PWR_FLAG"
-      (at 149.86 137.16 0)
-      (effects (font (size 1.27 1.27)) hide)
-    )
-    (property "Footprint" ""
-      (at 149.86 137.16 0)
-      (effects (font (size 1.27 1.27)) hide)
-    )
-    (property "Datasheet" ""
-      (at 149.86 137.16 0)
-      (effects (font (size 1.27 1.27)) hide)
-    )
-    (pin "1")
-  )
-  (wire
-    (pts (xy 149.86 137.16) (xy 149.86 139.70))
+    (pts (xy 149.86 134.62) (xy 149.86 139.70))
     (stroke (width 0) (type default))
   )
@@
     (on_board yes)
     (fields_autoplaced yes)
-    (property "Reference" "#PWR04"
+    (property "Reference" "#PWR303"
       (at 149.86 139.70 0)
       (effects (font (size 1.27 1.27)) hide)
@@
     (on_board yes)
     (fields_autoplaced yes)
-    (property "Reference" "#PWR05"
+    (property "Reference" "#PWR304"
       (at 116.84 170.18 0)
       (effects (font (size 1.27 1.27)) hide)
@@
     (on_board yes)
     (fields_autoplaced yes)
-    (property "Reference" "#PWR06"
+    (property "Reference" "#PWR305"
       (at 144.78 153.67 0)
       (effects (font (size 1.27 1.27)) hide)
@@
     (on_board yes)
     (fields_autoplaced yes)
-    (property "Reference" "#PWR07"
+    (property "Reference" "#PWR306"
       (at 149.86 177.80 0)
       (effects (font (size 1.27 1.27)) hide)
@@
     (on_board yes)
     (fields_autoplaced yes)
-    (property "Reference" "#PWR08"
+    (property "Reference" "#PWR307"
       (at 116.84 208.28 0)
       (effects (font (size 1.27 1.27)) hide)
@@
     (on_board yes)
     (fields_autoplaced yes)
-    (property "Reference" "#PWR09"
+    (property "Reference" "#PWR308"
       (at 144.78 191.77 0)
       (effects (font (size 1.27 1.27)) hide)
@@
     (on_board yes)
     (fields_autoplaced yes)
-    (property "Reference" "#PWR10"
+    (property "Reference" "#PWR309"
       (at 149.86 215.90 0)
       (effects (font (size 1.27 1.27)) hide)
@@
         (justify left top))
   )
-  (symbol
-    (lib_id "power:VCC")
-    (at 190.50 127.00 0)
-    (unit 1)
-    (exclude_from_sim no)
-    (in_bom yes)
-    (on_board yes)
-    (fields_autoplaced yes)
-    (property "Reference" "#PWR11"
-      (at 190.50 127.00 0)
-      (effects (font (size 1.27 1.27)) hide)
-    )
-    (property "Value" "+3V3"
-      (at 190.50 123.19 0)
-      (effects
-        (font
-          (size 1.27 1.27)
-        ))
-    )
-    (property "Footprint" ""
-      (at 190.50 127.00 0)
-      (effects (font (size 1.27 1.27)) hide)
-    )
-    (property "Datasheet" ""
-      (at 190.50 127.00 0)
-      (effects (font (size 1.27 1.27)) hide)
-    )
-    (pin "1")
-  )
-  (wire
-    (pts (xy 190.50 127.00) (xy 190.50 132.08))
-    (stroke (width 0) (type default))
-  )
-  (symbol
-    (lib_id "power:PWR_FLAG")
-    (at 190.50 132.08 0)
-    (unit 1)
-    (exclude_from_sim no)
-    (in_bom yes)
-    (on_board yes)
-    (fields_autoplaced yes)
-    (property "Reference" "#PWR12"
-      (at 190.50 132.08 0)
-      (effects (font (size 1.27 1.27)) hide)
-    )
-    (property "Value" "PWR_FLAG"
-      (at 190.50 132.08 0)
-      (effects (font (size 1.27 1.27)) hide)
-    )
-    (property "Footprint" ""
-      (at 190.50 132.08 0)
-      (effects (font (size 1.27 1.27)) hide)
-    )
-    (property "Datasheet" ""
-      (at 190.50 132.08 0)
-      (effects (font (size 1.27 1.27)) hide)
-    )
-    (pin "1")
-  )
-  (text "rail flag: driver on power sheet"
+  (text "+3V3/GND join by name; drivers on power sheet"
     (at 181.61 137.16 0)
     (effects

Commit message: layout: placed+silk+parity-0 (drc10: 0 errors/0 parity, 125 warnings)
Parts:
- SW401, SW402, SW403: footprint (none) -> trackball:D2FC-F-7N
Changed lines of the file:
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@@
         ))
     )
-    (property "Footprint" ""
+    (property "Description" "Omron D2FC-F-7N microswitch"
+    	(id 4)
+    	(at 0 0 0)
+    	(effects (font (size 1.27 1.27)) hide)
+    )
+    (property "Footprint" "trackball:D2FC-F-7N"
       (at 127.00 127.00 0)
       (effects (font (size 1.27 1.27)) hide)
     )
-    (property "Datasheet" ""
+    (property "Datasheet" "Omron D2F/D2FC series"
       (at 127.00 127.00 0)
       (effects (font (size 1.27 1.27)) hide)
@@
         ))
     )
-    (property "Footprint" ""
+    (property "Description" "Omron D2FC-F-7N microswitch"
+    	(id 4)
+    	(at 0 0 0)
+    	(effects (font (size 1.27 1.27)) hide)
+    )
+    (property "Footprint" "trackball:D2FC-F-7N"
       (at 127.00 165.10 0)
       (effects (font (size 1.27 1.27)) hide)
     )
-    (property "Datasheet" ""
+    (property "Datasheet" "Omron D2F/D2FC series"
       (at 127.00 165.10 0)
       (effects (font (size 1.27 1.27)) hide)
@@
         ))
     )
-    (property "Footprint" ""
+    (property "Description" "Omron D2FC-F-7N microswitch"
+    	(id 4)
+    	(at 0 0 0)
+    	(effects (font (size 1.27 1.27)) hide)
+    )
+    (property "Footprint" "trackball:D2FC-F-7N"
       (at 127.00 203.20 0)
       (effects (font (size 1.27 1.27)) hide)
     )
-    (property "Datasheet" ""
+    (property "Datasheet" "Omron D2F/D2FC series"
       (at 127.00 203.20 0)
       (effects (font (size 1.27 1.27)) hide)

Commit message: WIP routing drc143: unc 57, 0 viol, VBUS12/GND11
Connections:
- net Net-(SW401-NO): now reaches R401.1, SW401.2 (NO)
- net Net-(SW403-NO): now reaches R405.1, SW403.2 (NO)
- net Net-(SW402-NO): now reaches R403.1, SW402.2 (NO)
Changed lines of the file:
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@@
     (color 0 0 0 0)
   )
+  (label "Net-(SW401-NO)"
+    (at 134.62 127.00 0)
+    (effects
+        (font
+          (size 1.27 1.27)
+        )
+        (justify left bottom))
+  )
+  (label "Net-(SW402-NO)"
+    (at 134.62 165.10 0)
+    (effects
+        (font
+          (size 1.27 1.27)
+        )
+        (justify left bottom))
+  )
+  (label "Net-(SW403-NO)"
+    (at 134.62 203.20 0)
+    (effects
+        (font
+          (size 1.27 1.27)
+        )
+        (justify left bottom))
+  )
 )
