File: trackball-base/mcu.kicad_sch (KiCad schematic)
At the start: 19 parts, among them J201 TYPE-C-31-M-12, J202 CORTEX-DBG-10, SW201 RESET, SW202 BOOT, U201 E73-2G4M08S1C, U202 TPD2E1B06DRLR, Y201 ABS07-32.768KHZ-9-T

Commit message: base schematic complete: root + 5 sheets ERC-clean, review notes + BOM draft
Full hierarchical project (root + power/mcu/sensors/buttons/tx):
0 ERC errors, 1 benign pin_to_pin warning (ADC rail-sense, documented).
Netlist-verified: 145 comps, VSEN_1V9/MCU_RST/USB/SPI/TX nets.
Adds notes/SCHEMATIC_REVIEW.md (decisions, rail design, TX tree,
antenna, GPIO map, provisionals, ERC log) + notes/BOM_DRAFT.md.
Parts:
- added C207: 10uF/10V, Capacitor_SMD:C_0805_2012Metric, symbol Device:C_Small
- added C208: 4.7nF, Capacitor_SMD:C_0603_1608Metric, symbol Device:C_Small
- added R205: 1M, Resistor_SMD:R_0603_1608Metric, symbol Device:R_Small_US
- added R206, R207: 33, Resistor_SMD:R_0603_1608Metric, symbol Device:R_Small_US
- added TP203: TP203, TestPoint:TestPoint_Pad_D1.5mm, symbol Connector:TestPoint
- added TP204: TP204, TestPoint:TestPoint_Pad_D1.5mm, symbol Connector:TestPoint
- added TP205: TP205, TestPoint:TestPoint_Pad_D1.5mm, symbol Connector:TestPoint
- added TP206: TP206, TestPoint:TestPoint_Pad_D1.5mm, symbol Connector:TestPoint
- C203, C204: footprint Capacitor_SMD:C_0603_1608Metric -> Capacitor_SMD:C_0402_1005Metric
Connections:
- net +3V3: now also C207.1
- net GND: now also C207.2, C208.2, R205.2, TP206.1; no longer J201.SH (SHIELD)
- net MCU_RST: now also TP205.1
- net S1_SCK: now also R206.2; no longer U201.33 (P0.13)
- net S2_SCK: now also R207.1; no longer U201.20 (P0.12)
- net at J202.2 (Pin_2), U201.37 (SWDIO): now also TP203.1
- net at J202.4 (Pin_4), U201.39 (SWDCLK): now also TP204.1
- new net: R206.1, U201.33 (P0.13)
- new net: R207.2, U201.20 (P0.12)
- new net CHASSIS: C208.1, J201.SH (SHIELD), R205.1
Other:
- note added: "4. Unused nRF GPIOs P1.10/P0.26/P0.06/P0.08 + NFC P0.09/P0.10: NC on schematic,"
- note added: "FW configures input-with-pull, never hard-tied (ELEC-020). Antenna keepout under E73 end (layout)."
- note removed: "4. P0.09/P0.10 NFC pins unused; antenna keepout under E73 antenna end (layout)."

Commit message: layout: placed+silk+parity-0 (drc10: 0 errors/0 parity, 125 warnings)
Parts:
- added D203: ESD5Z5.0T1G, Diode_SMD:D_SOD-523, symbol Device:D_Schottky
- TP203, TP204, TP205, TP206: footprint TestPoint:TestPoint_Pad_D1.5mm -> TestPoint:TestPoint_Pad_D2.0mm
- U201: footprint (none) -> trackball:E73-2G4M08S1C
Connections:
- net GND: now also D203.2 (A)
- net VBUS: now also D203.1 (K)
Changed lines of the file:
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@@
         ))
     )
-    (property "Footprint" ""
+    (property "Description" "EBYTE E73-2G4M08S1C nRF52840 BLE module"
+    	(id 4)
+    	(at 0 0 0)
+    	(effects (font (size 1.27 1.27)) hide)
+    )
+    (property "Footprint" "trackball:E73-2G4M08S1C"
       (at 190.50 190.50 0)
       (effects (font (size 1.27 1.27)) hide)
     )
-    (property "Datasheet" ""
+    (property "Datasheet" "https://www.cdebyte.com/products/E73-2G4M08S1C"
       (at 190.50 190.50 0)
       (effects (font (size 1.27 1.27)) hide)
@@
         ))
     )
-    (property "Footprint" "TestPoint:TestPoint_Pad_D1.5mm"
+    (property "Footprint" "TestPoint:TestPoint_Pad_D2.0mm"
       (at 350.52 214.63 0)
       (effects (font (size 1.27 1.27)) hide)
@@
         ))
     )
-    (property "Footprint" "TestPoint:TestPoint_Pad_D1.5mm"
+    (property "Footprint" "TestPoint:TestPoint_Pad_D2.0mm"
       (at 248.92 210.82 0)
       (effects (font (size 1.27 1.27)) hide)
@@
         ))
     )
-    (property "Footprint" "TestPoint:TestPoint_Pad_D1.5mm"
+    (property "Footprint" "TestPoint:TestPoint_Pad_D2.0mm"
       (at 251.46 215.90 0)
       (effects (font (size 1.27 1.27)) hide)
@@
         ))
     )
-    (property "Footprint" "TestPoint:TestPoint_Pad_D1.5mm"
+    (property "Footprint" "TestPoint:TestPoint_Pad_D2.0mm"
       (at 299.72 212.09 0)
       (effects (font (size 1.27 1.27)) hide)
@@
     (color 0 0 0 0)
   )
+  (symbol
+    (lib_id "Device:D_Schottky")
+    (at 320.04 172.72 90)
+    (unit 1)
+    (exclude_from_sim no)
+    (in_bom yes)
+    (on_board yes)
+    (fields_autoplaced yes)
+    (property "Reference" "D203"
+      (at 326.39 168.91 0)
+      (effects
+        (font
+          (size 1.27 1.27)
+        ))
+    )
+    (property "Value" "ESD5Z5.0T1G"
+      (at 327.66 172.72 0)
+      (effects
+        (font
+          (size 1.27 1.27)
+        ))
+    )
+    (property "Footprint" "Diode_SMD:D_SOD-523"
+      (at 320.04 172.72 0)
+      (effects (font (size 1.27 1.27)) hide)
+    )
+    (property "Datasheet" "https://www.onsemi.com/pdf/datasheet/esd5z2v5t1-d.pdf"
+      (at 320.04 172.72 0)
+      (effects (font (size 1.27 1.27)) hide)
+    )
+    (pin "1")
+    (pin "2")
+  )
+  (wire
+    (pts (xy 320.04 167.64) (xy 320.04 168.91))
+    (stroke (width 0) (type default))
+  )
+  (wire
+    (pts (xy 320.04 176.53) (xy 322.58 176.53))
+    (stroke (width 0) (type default))
+  )
+  (global_label "VBUS"
+    (shape bidirectional)
+    (at 322.58 176.53 180)
+    (fields_autoplaced yes)
+    (effects
+        (font
+          (size 1.27 1.27)
+        ))
+    (property "Intersheetrefs" "${INTERSHEET_REFS}"
+      (at 322.58 176.53 180)
+      (effects (font (size 1.27 1.27)) hide)
+    )
+  )
+  (symbol
+    (lib_id "power:GND")
+    (at 320.04 167.64 0)
+    (unit 1)
+    (exclude_from_sim no)
+    (in_bom yes)
+    (on_board yes)
+    (fields_autoplaced yes)
+    (property "Reference" "#PWR509"
+      (at 320.04 167.64 0)
+      (effects (font (size 1.27 1.27)) hide)
+    )
+    (property "Value" "GND"
+      (at 320.04 167.64 0)
+      (effects (font (size 1.27 1.27)) hide)
+    )
+    (property "Footprint" ""
+      (at 320.04 167.64 0)
+      (effects (font (size 1.27 1.27)) hide)
+    )
+    (property "Datasheet" ""
+      (at 320.04 167.64 0)
+      (effects (font (size 1.27 1.27)) hide)
+    )
+    (pin "1")
+  )
 )

Commit message: WIP routing drc143: unc 57, 0 viol, VBUS12/GND11
Connections:
- net Net-(U201-P0.01/XL2): now reaches C202.1, U201.13 (P0.01/XL2), Y201.1
- net Net-(U201-P0.00/XL1): now reaches C201.2, U201.11 (P0.00/XL1), Y201.2
- net Net-(J202-Pin_2): now reaches J202.2 (Pin_2), TP203.1, U201.37 (SWDIO)
- net Net-(J202-Pin_4): now reaches J202.4 (Pin_4), TP204.1, U201.39 (SWDCLK)
- net Net-(U201-P0.28/AIN4): now reaches TP201.1, U201.4 (P0.28/AIN4)
- net Net-(U201-P0.29/AIN5): now reaches TP202.1, U201.8 (P0.29/AIN5)
- net Net-(U202-IOA1): now reaches J201.A7 (D-), J201.B7 (D-), U202.1 (IOA1)
- net Net-(U202-IOB1): now reaches J201.A6 (D+), J201.B6 (D+), U202.2 (IOB1)
- net Net-(U201-D+): now reaches U201.31 (D+), U202.4 (IOB2)
- net Net-(U201-D-): now reaches U201.29 (D-), U202.5 (IOA2)
- net Net-(J201-CC1): now reaches J201.A5 (CC1), R203.2
- net Net-(U201-P0.13): now reaches R206.1, U201.33 (P0.13)
- net Net-(U201-P1.11): now reaches R201.2, SW202.2, U201.1 (P1.11)
- net Net-(U201-P0.12): now reaches R207.2, U201.20 (P0.12)
- net Net-(J201-CC2): now reaches J201.B5 (CC2), R204.1
Changed lines of the file:
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@@
     (pin "1")
   )
+  (label "Net-(J201-CC1)"
+    (at 292.10 123.19 0)
+    (effects
+        (font
+          (size 1.27 1.27)
+        )
+        (justify left bottom))
+  )
+  (label "Net-(J201-CC2)"
+    (at 342.90 123.19 0)
+    (effects
+        (font
+          (size 1.27 1.27)
+        )
+        (justify left bottom))
+  )
+  (label "Net-(J202-Pin_2)"
+    (at 325.12 204.47 0)
+    (effects
+        (font
+          (size 1.27 1.27)
+        )
+        (justify left bottom))
+  )
+  (label "Net-(J202-Pin_4)"
+    (at 325.12 207.01 0)
+    (effects
+        (font
+          (size 1.27 1.27)
+        )
+        (justify left bottom))
+  )
+  (label "Net-(U201-D+)"
+    (at 207.01 185.42 0)
+    (effects
+        (font
+          (size 1.27 1.27)
+        )
+        (justify left bottom))
+  )
+  (label "Net-(U201-D-)"
+    (at 207.01 180.34 0)
+    (effects
+        (font
+          (size 1.27 1.27)
+        )
+        (justify left bottom))
+  )
+  (label "Net-(U201-P0.00{slash}XL1)"
+    (at 137.16 190.50 0)
+    (effects
+        (font
+          (size 1.27 1.27)
+        )
+        (justify left bottom))
+  )
+  (label "Net-(U201-P0.01{slash}XL2)"
+    (at 130.81 193.04 0)
+    (effects
+        (font
+          (size 1.27 1.27)
+        )
+        (justify left bottom))
+  )
+  (label "Net-(U201-P0.12)"
+    (at 168.91 212.09 0)
+    (effects
+        (font
+          (size 1.27 1.27)
+        )
+        (justify left bottom))
+  )
+  (label "Net-(U201-P0.13)"
+    (at 215.90 190.50 0)
+    (effects
+        (font
+          (size 1.27 1.27)
+        )
+        (justify left bottom))
+  )
+  (label "Net-(U201-P0.28{slash}AIN4)"
+    (at 165.10 167.64 90)
+    (effects
+        (font
+          (size 1.27 1.27)
+        )
+        (justify left bottom))
+  )
+  (label "Net-(U201-P0.29{slash}AIN5)"
+    (at 142.24 179.07 90)
+    (effects
+        (font
+          (size 1.27 1.27)
+        )
+        (justify left bottom))
+  )
+  (label "Net-(U201-P1.11)"
+    (at 165.10 160.02 90)
+    (effects
+        (font
+          (size 1.27 1.27)
+        )
+        (justify left bottom))
+  )
+  (label "Net-(U202-IOA1)"
+    (at 302.26 128.27 0)
+    (effects
+        (font
+          (size 1.27 1.27)
+        )
+        (justify left bottom))
+  )
+  (label "Net-(U202-IOB1)"
+    (at 302.26 125.73 0)
+    (effects
+        (font
+          (size 1.27 1.27)
+        )
+        (justify left bottom))
+  )
 )
