File: trackball-base/power.kicad_sch (KiCad schematic)
At the start: 44 parts, among them Q101 2N7002, U101 AP2112K-3.3TRG1, U102 APX809-29SAG-7, U103 XC6206P192MR, U104 TPS22918DBVR, U105 TPS22918DBVR, U106 TLV3011AIDBVR, U107 TLV3011AIDBVR

Commit message: layout: placed+silk+parity-0 (drc10: 0 errors/0 parity, 125 warnings)
Connections:
- net GND: now also Q101.2 (S); no longer Q101.1 (S)
- net at R109.2, R110.2, U107.1 (OUT): now also Q101.1 (G); no longer Q101.2 (G)
Changed lines of the file:
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@@
       (effects (font (size 1.27 1.27)) hide)
     )
+    (pin "1")
+    (pin "3")
     (pin "2")
-    (pin "3")
-    (pin "1")
   )
   (wire

Commit message: WIP routing drc143: unc 57, 0 viol, VBUS12/GND11
Connections:
- net Net-(U107-IN+): now reaches R107.2, R108.1, R109.1, U107.3 (IN+)
- net Net-(Q101-G): now reaches Q101.1 (G), R109.2, R110.2, U107.1 (OUT)
- net Net-(U104-CT): now reaches C111.2, U104.4 (CT)
- net Net-(U105-CT): now reaches C116.2, U105.4 (CT)
- net Net-(U106-IN+): now reaches R104.2, R105.1, R106.1, U106.3 (IN+)
Changed lines of the file:
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@@
     (color 0 0 0 0)
   )
+  (label "Net-(Q101-G)"
+    (at 326.39 191.77 90)
+    (effects
+        (font
+          (size 1.27 1.27)
+        )
+        (justify left bottom))
+  )
+  (label "Net-(U104-CT)"
+    (at 185.42 124.46 0)
+    (effects
+        (font
+          (size 1.27 1.27)
+        )
+        (justify left bottom))
+  )
+  (label "Net-(U105-CT)"
+    (at 287.02 73.66 0)
+    (effects
+        (font
+          (size 1.27 1.27)
+        )
+        (justify left bottom))
+  )
+  (label "Net-(U106-IN+)"
+    (at 281.94 129.54 90)
+    (effects
+        (font
+          (size 1.27 1.27)
+        )
+        (justify left bottom))
+  )
+  (label "Net-(U107-IN+)"
+    (at 281.94 167.64 90)
+    (effects
+        (font
+          (size 1.27 1.27)
+        )
+        (justify left bottom))
+  )
 )

Commit message: Q5 ECO + pre-ripup checkpoint: R113/114/115/515 jumpers, drc129 33unc/0err/0parity
Schematic (owner-approved 2026-10-04): 3x 0R branch jumpers on power
sheet (R113 VBUS_SENSE, R114 SENSOR_EN, R115 MCU_TX_EN) + R515 CTD
in-line on tx (net split /tx/CTD_U501 + /tx/Net-(U501-CTD)). ERC 0
errors + 1 known benign warning; netlist diff minimal (4 nets only).
PCB: 4x 0603 staged, nets assigned, U501.14 on CTD_U501; 0 parity.
Docs: SCHEMATIC_REVIEW §11, BOM row, LAYOUT_REVIEW E53, QUESTIONS.
Reversible checkpoint before Q6 ripup.
Parts:
- added R113, R114, R115: 0R, Resistor_SMD:R_0603_1608Metric, symbol Device:R_Small_US
Connections:
- net MCU_TX_EN: now also R115.1, R115.2
- net SENSOR_EN: now also R114.1, R114.2
- net VBUS_SENSE: now also R113.1, R113.2
Other:
- note added: "Q5 jumper R113"
- note added: "Q5 jumper R114"
- note added: "Q5 jumper R115"
